File: pcb/counter/counter.kicad_pcb (KiCad board)
At the start: 2 copper layers, 82 x 32.4 mm, 22 parts, among them J1 Conn_01x01, J2 Conn_01x01, J3 Conn_01x01, J4 0.2", J5 0.2", J6 JST XH, J7 0.2", Q1 MMBT3904, U1 74HCT08

Commit message: Fill zones.
Routing:
- added copper zone on F.Cu, net +5V
- added copper zone on B.Cu, net GND
Changed lines of the file:
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@@
     (property "Sheetname" "")
     (attr through_hole)
-    (fp_text reference "J7" (at 14.224 -5.334 180) (layer "F.SilkS")
+    (fp_text reference "J7" (at 14.478 3.302 180) (layer "F.SilkS")
       (effects (font (size 1 1) (thickness 0.15)))
     )
@@
   (via (at 119.888 58.293) (size 0.8) (drill 0.4) (layers "F.Cu" "B.Cu") (net 20))
   (segment (start 124.968 58.293) (end 119.888 58.293) (width 0.25) (layer "B.Cu") (net 20))
+  (zone (net 3) (net_name "+5V") (layer "F.Cu") (hatch edge 0.508)
+    (connect_pads (clearance 0.508))
+    (min_thickness 0.254) (filled_areas_thickness no)
+    (fill yes (thermal_gap 0.508) (thermal_bridge_width 0.508))
+    (polygon
+      (pts
+        (xy 147.828 85.09)
+        (xy 104.14 85.09)
+        (xy 104.14 69.342)
+        (xy 147.828 69.342)
+      )
+    )
+  )
+  (zone (net 2) (net_name "GND") (layer "B.Cu") (hatch edge 0.508)
+    (connect_pads (clearance 0.508))
+    (min_thickness 0.254) (filled_areas_thickness no)
+    (fill yes (thermal_gap 0.508) (thermal_bridge_width 0.508))
+    (polygon
+      (pts
+        (xy 147.32 84.582)
+        (xy 103.886 84.582)
+        (xy 103.886 71.628)
+        (xy 98.298 66.294)
+        (xy 98.298 47.752)
+        (xy 147.32 47.752)
+      )
+    )
+  )
 )

Commit message: Order.
Other:
- rule pad_to_mask_clearance: 0.051 -> 0
Changed lines of the file:
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@@
   )
   (paper "A4")
+  (title_block
+    (comment 4 "AISLER Project ID: SVPGSVLX")
+  )
   (layers
     (0 "F.Cu" signal)
@@
   )
   (setup
-    (pad_to_mask_clearance 0.051)
-    (solder_mask_min_width 0.25)
+    (pad_to_mask_clearance 0)
     (pcbplotparams
       (layerselection 0x00030fc_ffffffff)
@@
     (fp_line (start -2.65 -2.15) (end -3.65 -1.15) (layer "F.Fab") (width 0.1))
     (fp_line (start -3.65 2.15) (end 3.65 2.15) (layer "F.Fab") (width 0.1))
-    (pad "1" smd roundrect (at -3.1125 0) (size 2.075 2.55) (layers "F.Cu" "F.Paste" "F.Mask") (roundrect_rratio 0.120482)
+    (pad "1" smd roundrect (at -3.1125 0) (size 2.075 2.55) (layers "F.Cu" "F.Paste" "F.Mask") (roundrect_rratio 0.1204819277)
       (net 3 "+5V") (pintype "passive"))
-    (pad "2" smd roundrect (at 3.1125 0) (size 2.075 2.55) (layers "F.Cu" "F.Paste" "F.Mask") (roundrect_rratio 0.120482)
+    (pad "2" smd roundrect (at 3.1125 0) (size 2.075 2.55) (layers "F.Cu" "F.Paste" "F.Mask") (roundrect_rratio 0.1204819277)
       (net 2 "GND") (pintype "passive"))
     (model "${KICAD6_3DMODEL_DIR}/Capacitor_Tantalum_SMD.3dshapes/CP_EIA-7343-40_Kemet-Y.wrl"
