File: pcb/counter/counter.kicad_pcb (KiCad board)
At the start: 2 copper layers, 82 x 32.4 mm, 22 parts, among them J1 Conn_01x01, J2 Conn_01x01, J3 Conn_01x01, J4 0.2", J5 0.2", J6 JST XH, J7 0.2", Q1 MMBT3904, U1 74HCT08

Commit message: Fix bug.
Connections:
- J4 pad 1: Net-(J4-Pad1) -> TH
- J4 pad 2: TH -> Net-(J4-Pad2)
- J6 pad 2: Net-(J4-Pad1) -> TH
- J6 pad 3: TH -> Net-(J4-Pad2)
- R4 pad 1: Net-(J4-Pad1) -> TH
- U1 pad 4: Net-(J4-Pad1) -> TH
- U1 pad 5: Net-(J4-Pad1) -> TH
Routing:
- net Net-(J4-Pad1): track 23.5 -> 0.00 mm
- net Net-(J4-Pad2): track 0.00 -> 10.7 mm
- net TH: track 22.2 -> 29.7 mm
Changed lines of the file:
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@@
   (net 8 "Net-(D2-Pad2)")
   (net 9 "Net-(J4-Pad3)")
-  (net 10 "Net-(J4-Pad1)")
+  (net 10 "Net-(J4-Pad2)")
   (net 11 "Net-(J4-Pad5)")
   (net 12 "Net-(J5-Pad1)")
@@
     (fp_line (start -2.5 2.55) (end 27.9 2.55) (layer "F.Fab") (width 0.1))
     (pad "1" thru_hole rect locked (at 0 0) (size 4 4) (drill 1.52) (layers *.Cu *.Mask)
-      (net 10 "Net-(J4-Pad1)") (pinfunction "Pin_1") (pintype "passive"))
+      (net 17 "TH") (pinfunction "Pin_1") (pintype "passive"))
     (pad "2" thru_hole circle locked (at 5.08 0) (size 4 4) (drill 1.52) (layers *.Cu *.Mask)
-      (net 17 "TH") (pinfunction "Pin_2") (pintype "passive"))
+      (net 10 "Net-(J4-Pad2)") (pinfunction "Pin_2") (pintype "passive"))
     (pad "3" thru_hole circle locked (at 10.16 0) (size 4 4) (drill 1.52) (layers *.Cu *.Mask)
       (net 9 "Net-(J4-Pad3)") (pinfunction "Pin_3") (pintype "passive"))
@@
       (net 3 "+5V") (pinfunction "Pin_1") (pintype "passive"))
     (pad "2" thru_hole oval locked (at 2.5 0) (size 1.8 3) (drill 0.95) (layers *.Cu *.Mask)
-      (net 10 "Net-(J4-Pad1)") (pinfunction "Pin_2") (pintype "passive"))
+      (net 17 "TH") (pinfunction "Pin_2") (pintype "passive"))
     (pad "3" thru_hole oval locked (at 5 0) (size 1.8 3) (drill 0.95) (layers *.Cu *.Mask)
-      (net 17 "TH") (pinfunction "Pin_3") (pintype "passive"))
+      (net 10 "Net-(J4-Pad2)") (pinfunction "Pin_3") (pintype "passive"))
     (pad "4" thru_hole oval locked (at 7.5 0) (size 1.8 3) (drill 0.95) (layers *.Cu *.Mask)
       (net 9 "Net-(J4-Pad3)") (pinfunction "Pin_4") (pintype "passive"))
@@
       (net 15 "Net-(R3-Pad2)") (pintype "output"))
     (pad "4" smd roundrect (at -2.475 0 90) (size 1.95 0.6) (layers "F.Cu" "F.Paste" "F.Mask") (roundrect_rratio 0.25)
-      (net 10 "Net-(J4-Pad1)") (pintype "input"))
+      (net 17 "TH") (pintype "input"))
     (pad "5" smd roundrect (at -2.475 1.27 90) (size 1.95 0.6) (layers "F.Cu" "F.Paste" "F.Mask") (roundrect_rratio 0.25)
-      (net 10 "Net-(J4-Pad1)") (pintype "input"))
+      (net 17 "TH") (pintype "input"))
     (pad "6" smd roundrect (at -2.475 2.54 90) (size 1.95 0.6) (layers "F.Cu" "F.Paste" "F.Mask") (roundrect_rratio 0.25)
       (net 14 "Net-(R1-Pad2)") (pintype "output"))
@@
     (property "Sheetname" "")
     (attr through_hole)
-    (fp_text reference "J7" (at 14.224 -5.334 180) (layer "F.SilkS")
+    (fp_text reference "J7" (at 14.859 2.667 180) (layer "F.SilkS")
       (effects (font (size 1 1) (thickness 0.15)))
     )
@@
     (fp_line (start -0.8 0.4125) (end -0.8 -0.4125) (layer "F.Fab") (width 0.1))
     (pad "1" smd roundrect (at -0.825 0 180) (size 0.8 0.95) (layers "F.Cu" "F.Paste" "F.Mask") (roundrect_rratio 0.25)
-      (net 10 "Net-(J4-Pad1)") (pintype "passive"))
+      (net 17 "TH") (pintype "passive"))
     (pad "2" smd roundrect (at 0.825 0 180) (size 0.8 0.95) (layers "F.Cu" "F.Paste" "F.Mask") (roundrect_rratio 0.25)
       (net 2 "GND") (pintype "passive"))
@@
   (segment (start 124.968 69.596) (end 127 69.596) (width 0.5) (layer "B.Cu") (net 9))
   (segment (start 123.324 65.532) (end 123.324 67.532) (width 0.5) (layer "B.Cu") (net 9))
-  (segment (start 119.126 64.73) (end 118.324 65.532) (width 0.25) (layer "F.Cu") (net 10))
-  (segment (start 120.396 60.641) (end 119.126 60.641) (width 0.25) (layer "F.Cu") (net 10))
-  (segment (start 112.077 63.246) (end 116.24262 63.246) (width 0.25) (layer "F.Cu") (net 10))
-  (segment (start 118.324 65.32738) (end 118.324 65.532) (width 0.25) (layer "F.Cu") (net 10))
-  (segment (start 119.126 60.641) (end 119.126 64.73) (width 0.25) (layer "F.Cu") (net 10))
-  (segment (start 116.24262 63.246) (end 118.324 65.32738) (width 0.25) (layer "F.Cu") (net 10))
-  (segment (start 118.324 65.532) (end 118.324 75.144) (width 1.5) (layer "B.Cu") (net 10))
-  (segment (start 118.324 75.144) (end 118.364 75.184) (width 1.5) (layer "B.Cu") (net 10))
+  (segment (start 123.444 71.12) (end 123.444 75.184) (width 0.5) (layer "B.Cu") (net 10))
+  (segment (start 120.824 68.5) (end 120.824 65.532) (width 0.5) (layer "B.Cu") (net 10))
+  (segment (start 120.824 68.5) (end 123.444 71.12) (width 0.5) (layer "B.Cu") (net 10))
   (segment (start 138.684 75.184) (end 143.764 75.184) (width 0.5) (layer "B.Cu") (net 11))
   (segment (start 70.231 53.848) (end 69.215 52.832) (width 1) (layer "F.Cu") (net 12))
@@
   (segment (start 114.554 62.23) (end 117.348 62.23) (width 0.25) (layer "F.Cu") (net 15))
   (segment (start 128.333 61.722) (end 131.064 61.722) (width 0.25) (layer "F.Cu") (net 16))
-  (segment (start 121.666 55.691) (end 121.021 56.336) (width 0.25) (layer "F.Cu") (net 17))
-  (segment (start 121.021 65.335) (end 120.824 65.532) (width 0.25) (layer "F.Cu") (net 17))
+  (segment (start 119.126 64.73) (end 118.324 65.532) (width 0.25) (layer "F.Cu") (net 17))
+  (segment (start 120.396 55.691) (end 120.396 60.641) (width 0.25) (layer "F.Cu") (net 17))
+  (segment (start 120.396 60.641) (end 119.126 60.641) (width 0.25) (layer "F.Cu") (net 17))
+  (segment (start 112.077 63.246) (end 116.24262 63.246) (width 0.25) (layer "F.Cu") (net 17))
+  (segment (start 118.324 65.32738) (end 118.324 65.532) (width 0.25) (layer "F.Cu") (net 17))
   (segment (start 120.396 55.691) (end 121.666 55.691) (width 0.25) (layer "F.Cu") (net 17))
-  (segment (start 121.021 56.336) (end 121.021 65.335) (width 0.25) (layer "F.Cu") (net 17))
-  (segment (start 123.444 71.12) (end 123.444 75.184) (width 0.5) (layer "B.Cu") (net 17))
-  (segment (start 120.824 68.5) (end 123.444 71.12) (width 0.5) (layer "B.Cu") (net 17))
-  (segment (start 120.824 65.532) (end 120.824 68.5) (width 0.5) (layer "B.Cu") (net 17))
+  (segment (start 119.126 60.641) (end 119.126 64.73) (width 0.25) (layer "F.Cu") (net 17))
+  (segment (start 116.24262 63.246) (end 118.324 65.32738) (width 0.25) (layer "F.Cu") (net 17))
+  (segment (start 118.324 65.532) (end 118.324 75.144) (width 1.5) (layer "B.Cu") (net 17))
+  (segment (start 118.324 75.144) (end 118.364 75.184) (width 1.5) (layer "B.Cu") (net 17))
   (segment (start 105.8395 61.656) (end 107.567 61.656) (width 0.25) (layer "F.Cu") (net 18))
   (segment (start 107.567 61.656) (end 107.633 61.722) (width 0.25) (layer "F.Cu") (net 18))
@@
   (segment (start 137.097 61.722) (end 131.066 55.691) (width 0.25) (layer "F.Cu") (net 19))
   (segment (start 126.683 61.722) (end 126.683 60.008) (width 0.25) (layer "F.Cu") (net 20))
-  (segment (start 119.888 58.293) (end 119.126 57.531) (width 0.25) (layer "F.Cu") (net 20))
+  (segment (start 119.126 55.691) (end 119.126 57.836987) (width 0.25) (layer "F.Cu") (net 20))
+  (segment (start 119.126 57.836987) (end 119.6715 58.382487) (width 0.25) (layer "F.Cu") (net 20))
   (segment (start 126.683 60.008) (end 124.968 58.293) (width 0.25) (layer "F.Cu") (net 20))
-  (segment (start 119.126 57.531) (end 119.126 55.691) (width 0.25) (layer "F.Cu") (net 20))
   (via (at 124.968 58.293) (size 0.8) (drill 0.4) (layers "F.Cu" "B.Cu") (net 20))
-  (via (at 119.888 58.293) (size 0.8) (drill 0.4) (layers "F.Cu" "B.Cu") (net 20))
+  (via (at 119.6715 58.382487) (size 0.8) (drill 0.4) (layers "F.Cu" "B.Cu") (net 20))
+  (segment (start 119.798513 58.382487) (end 119.6715 58.382487) (width 0.25) (layer "B.Cu") (net 20))
+  (segment (start 119.888 58.293) (end 119.798513 58.382487) (width 0.25) (layer "B.Cu") (net 20))
   (segment (start 124.968 58.293) (end 119.888 58.293) (width 0.25) (layer "B.Cu") (net 20))
 )
