File: pcb/counter/counter.kicad_sch (KiCad schematic)
At the start: 19 parts, among them J1 Conn_01x01, J2 Conn_01x01, J3 Conn_01x01, J4 0.2", J5 0.2", J6 JST XH, J7 0.2", Q1 Q_NPN_CBE, U1 74HC08

Commit message: Update footprints for SMD version.
Parts:
- added R5: 820, Resistor_SMD:R_0201_0603Metric, symbol Device:R
- added R6: 820, Capacitor_Tantalum_SMD:CP_EIA-7343-40_Kemet-Y, symbol Device:R
- C1: value 1u -> 10u; footprint Capacitor_THT:C_Rect_L11.0mm_W7.3mm_P10.00mm_MKT -> Capacitor_SMD:C_0805_2012Metric
- C2: footprint Capacitor_THT:CP_Radial_D10.0mm_P2.50mm_P5.00mm -> Capacitor_Tantalum_SMD:CP_EIA-7343-40_Kemet-Y
- D1: footprint Diode_THT:D_DO-41_SOD81_P10.16mm_Horizontal -> Diode_SMD:D_MiniMELF
- D2, D3: renamed from D?; footprint (none) -> LED_THT:LED_D5.0mm_Horizontal_O1.27mm_Z3.0mm
- Q1: value Q_NPN_CBE -> MMBT3904; footprint Package_TO_SOT_THT:TO-92L_Wide -> Package_TO_SOT_SMD:SOT-23; symbol Device:Q_NPN_CBE -> Transistor_BJT:BC849
- R1, R3: footprint Resistor_THT:R_Axial_DIN0411_L9.9mm_D3.6mm_P12.70mm_Horizontal -> Resistor_SMD:R_0201_0603Metric
- R2: footprint Resistor_THT:R_Axial_DIN0411_L9.9mm_D3.6mm_P5.08mm_Vertical -> Resistor_SMD:R_0201_0603Metric
- R4: footprint Resistor_THT:R_Axial_DIN0411_L9.9mm_D3.6mm_P7.62mm_Vertical -> Resistor_SMD:R_0201_0603Metric
- U1: value 74HC08 -> 74HCT08; footprint Package_DIP:DIP-14_W7.62mm_LongPads -> Package_SO:SOIC-14_3.9x8.7mm_P1.27mm
- gave numbers to parts that had none: 1
Connections:
- net +5V: no longer U1.12, U1.13
- net GND: now also D2.1 (K), D3.1 (K), Q1.2 (E); no longer Q1.3 (E), U1.10, U1.9
- net RELAY: now also Q1.3 (C); no longer Q1.1 (C)
- net TH: now reaches J4.2 (Pin_2), J6.3 (Pin_3)
- net TH: now also U1.10, U1.9
- net at C1.1, D1.1 (K), R2.1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: now also U1.12, U1.13
- net at R3.1: now also Q1.1 (B); no longer Q1.2 (B)
- net at U1.8: now also R5.1
- net at U1.11: now also R6.1
- net at D3.2 (A): now also R6.2
- net at D2.2 (A): now also R5.2
- no-connect marks 2 -> 0
Other:
- note added: "230 V out"
- note added: "Laser enable"
- note added: "PWM"
- moved on the sheet: C2, D2, D3, U1D

Commit message: Add protection diode; work on routing.
Parts:
- added D4: 1N4148, Diode_SMD:D_MiniMELF, symbol Device:D
- R1, R2, R3, R4, R5: footprint Resistor_SMD:R_0201_0603Metric -> Resistor_SMD:R_0603_1608Metric
- R6: footprint Capacitor_Tantalum_SMD:CP_EIA-7343-40_Kemet-Y -> Resistor_SMD:R_0603_1608Metric
Connections:
- net GND: now also D4.2 (A)
- net RELAY: now also D4.1 (K)
- net at J4.1 (Pin_1), J6.2 (Pin_2), R4.1: now also U1.4, U1.5; no longer U1.1, U1.2
- net at R1.2: now also U1.6; no longer U1.3
- net at C1.1, D1.1 (K), R2.1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: now also U1.1, U1.2; no longer U1.4, U1.5
- net at R3.2: now also U1.3; no longer U1.6
Changed lines of the file:
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@@
   (junction (at 52.07 52.07) (diameter 0) (color 0 0 0 0)
   )
+  (junction (at 177.165 90.17) (diameter 0) (color 0 0 0 0)
+  )
   (junction (at 57.15 95.25) (diameter 0) (color 0 0 0 0)
   )
   (junction (at 49.53 48.26) (diameter 0) (color 0 0 0 0)
   )
+  (junction (at 160.02 107.95) (diameter 0) (color 0 0 0 0)
+  )
   (junction (at 121.92 95.25) (diameter 0) (color 0 0 0 0)
   )
@@
     (stroke (width 0) (type default) (color 0 0 0 0))
   )
+  (wire (pts (xy 177.165 107.95) (xy 177.165 102.235))
+    (stroke (width 0) (type default) (color 0 0 0 0))
+  )
   (wire (pts (xy 57.15 100.33) (xy 63.5 100.33))
     (stroke (width 0) (type default) (color 0 0 0 0))
@@
     (stroke (width 0) (type default) (color 0 0 0 0))
   )
+  (wire (pts (xy 160.02 107.95) (xy 177.165 107.95))
+    (stroke (width 0) (type default) (color 0 0 0 0))
+  )
   (wire (pts (xy 78.74 163.195) (xy 78.74 165.735))
     (stroke (width 0) (type default) (color 0 0 0 0))
@@
     (stroke (width 0) (type default) (color 0 0 0 0))
   )
+  (wire (pts (xy 177.165 90.17) (xy 177.165 94.615))
+    (stroke (width 0) (type default) (color 0 0 0 0))
+  )
   (wire (pts (xy 121.92 62.23) (xy 125.095 62.23))
     (stroke (width 0) (type default) (color 0 0 0 0))
@@
     (stroke (width 0) (type default) (color 0 0 0 0))
   )
+  (wire (pts (xy 177.165 90.17) (xy 183.515 90.17))
+    (stroke (width 0) (type default) (color 0 0 0 0))
+  )
   (wire (pts (xy 78.74 143.51) (xy 78.74 146.685))
     (stroke (width 0) (type default) (color 0 0 0 0))
@@
     (stroke (width 0) (type default) (color 0 0 0 0))
   )
-  (wire (pts (xy 163.83 90.17) (xy 160.02 90.17))
+  (wire (pts (xy 160.02 90.17) (xy 177.165 90.17))
     (stroke (width 0) (type default) (color 0 0 0 0))
   )
@@
     )
   )
-  (global_label "RELAY" (shape input) (at 163.83 90.17 0) (fields_autoplaced)
+  (global_label "RELAY" (shape input) (at 183.515 90.17 0) (fields_autoplaced)
     (effects (font (size 1.27 1.27)) (justify left))
-    (property "Intersheet References" "${INTERSHEET_REFS}" (id 0) (at 250.19 -69.85 0)
+    (property "Intersheet References" "${INTERSHEET_REFS}" (id 0) (at 269.875 -69.85 0)
       (effects (font (size 1.27 1.27)) hide)
     )
@@
     (pin "8")
   )
-  (symbol (lib_name "74LS08_2") (lib_id "74xx:74LS08") (at 71.12 97.79 0) (unit 1)
+  (symbol (lib_name "74LS08_2") (lib_id "74xx:74LS08") (at 71.12 97.79 0) (unit 2)
     (in_bom yes) (on_board yes)
     (property "Reference" "U1" (id 0) (at 71.12 89.535 0))
@@
     (property "Reference" "R1" (id 0) (at 86.36 92.5322 90))
     (property "Value" "100" (id 1) (at 86.36 94.8436 90))
-    (property "Footprint" "Resistor_SMD:R_0201_0603Metric" (id 2) (at 86.36 96.012 90)
+    (property "Footprint" "Resistor_SMD:R_0603_1608Metric" (id 2) (at 86.36 96.012 90)
       (effects (font (size 1.27 1.27)) hide)
     )
@@
       (effects (font (size 1.27 1.27)) (justify left))
     )
-    (property "Footprint" "Resistor_SMD:R_0201_0603Metric" (id 2) (at 115.062 102.87 90)
+    (property "Footprint" "Resistor_SMD:R_0603_1608Metric" (id 2) (at 115.062 102.87 90)
       (effects (font (size 1.27 1.27)) hide)
     )
@@
     (pin "2")
   )
-  (symbol (lib_name "74LS08_4") (lib_id "74xx:74LS08") (at 132.08 97.79 0) (unit 2)
+  (symbol (lib_name "74LS08_4") (lib_id "74xx:74LS08") (at 132.08 97.79 0) (unit 1)
     (in_bom yes) (on_board yes)
     (property "Reference" "U1" (id 0) (at 132.08 89.535 0))
@@
     (property "Reference" "R3" (id 0) (at 146.05 92.5322 90))
     (property "Value" "1k" (id 1) (at 146.05 94.8436 90))
-    (property "Footprint" "Resistor_SMD:R_0201_0603Metric" (id 2) (at 146.05 96.012 90)
+    (property "Footprint" "Resistor_SMD:R_0603_1608Metric" (id 2) (at 146.05 96.012 90)
       (effects (font (size 1.27 1.27)) hide)
     )
@@
       (effects (font (size 1.27 1.27)) (justify left))
     )
-    (property "Footprint" "Resistor_SMD:R_0201_0603Metric" (id 2) (at 55.372 106.68 90)
+    (property "Footprint" "Resistor_SMD:R_0603_1608Metric" (id 2) (at 55.372 106.68 90)
       (effects (font (size 1.27 1.27)) hide)
     )
@@
     (property "Reference" "R6" (id 0) (at 146.05 58.42 90))
     (property "Value" "820" (id 1) (at 146.05 60.96 90))
-    (property "Footprint" "Capacitor_Tantalum_SMD:CP_EIA-7343-40_Kemet-Y" (id 2) (at 146.05 66.548 90)
+    (property "Footprint" "Resistor_SMD:R_0603_1608Metric" (id 2) (at 146.05 66.548 90)
       (effects (font (size 1.27 1.27)) hide)
     )
@@
       (effects (font (size 1.27 1.27)) (justify left))
     )
-    (property "Footprint" "Resistor_SMD:R_0201_0603Metric" (id 2) (at 76.962 150.495 90)
+    (property "Footprint" "Resistor_SMD:R_0603_1608Metric" (id 2) (at 76.962 150.495 90)
       (effects (font (size 1.27 1.27)) hide)
     )
     (property "Datasheet" "~" (id 3) (at 78.74 150.495 0)
+      (effects (font (size 1.27 1.27)) hide)
+    )
+    (pin "1")
+    (pin "2")
+  )
+  (symbol (lib_id "Device:D") (at 177.165 98.425 270) (unit 1)
+    (in_bom yes) (on_board yes) (fields_autoplaced)
+    (property "Reference" "D4" (id 0) (at 180.34 97.1549 90)
+      (effects (font (size 1.27 1.27)) (justify left))
+    )
+    (property "Value" "1N4148" (id 1) (at 180.34 99.6949 90)
+      (effects (font (size 1.27 1.27)) (justify left))
+    )
+    (property "Footprint" "Diode_SMD:D_MiniMELF" (id 2) (at 177.165 98.425 0)
+      (effects (font (size 1.27 1.27)) hide)
+    )
+    (property "Datasheet" "~" (id 3) (at 177.165 98.425 0)
       (effects (font (size 1.27 1.27)) hide)
     )
@@
       (reference "D3") (unit 1) (value "LED") (footprint "LED_THT:LED_D5.0mm_Horizontal_O1.27mm_Z3.0mm")
     )
+    (path "/92441e7a-5980-432c-8910-40637e2ef2b6"
+      (reference "D4") (unit 1) (value "1N4148") (footprint "Diode_SMD:D_MiniMELF")
+    )
     (path "/00000000-0000-0000-0000-00005dff8675"
       (reference "J1") (unit 1) (value "Conn_01x01") (footprint "Connector_Pin:Pin_D1.0mm_L10.0mm")
@@
     )
     (path "/00000000-0000-0000-0000-00005dfd2ef8"
-      (reference "R1") (unit 1) (value "100") (footprint "Resistor_SMD:R_0201_0603Metric")
+      (reference "R1") (unit 1) (value "100") (footprint "Resistor_SMD:R_0603_1608Metric")
     )
     (path "/00000000-0000-0000-0000-00005dfd5b1d"
-      (reference "R2") (unit 1) (value "1M") (footprint "Resistor_SMD:R_0201_0603Metric")
+      (reference "R2") (unit 1) (value "1M") (footprint "Resistor_SMD:R_0603_1608Metric")
     )
     (path "/00000000-0000-0000-0000-00005dfdb71c"
-      (reference "R3") (unit 1) (value "1k") (footprint "Resistor_SMD:R_0201_0603Metric")
+      (reference "R3") (unit 1) (value "1k") (footprint "Resistor_SMD:R_0603_1608Metric")
     )
     (path "/00000000-0000-0000-0000-00005e034112"
-      (reference "R4") (unit 1) (value "100k") (footprint "Resistor_SMD:R_0201_0603Metric")
+      (reference "R4") (unit 1) (value "100k") (footprint "Resistor_SMD:R_0603_1608Metric")
     )
     (path "/7b39b144-f043-4b61-b95e-acb320e64491"
-      (reference "R5") (unit 1) (value "820") (footprint "Resistor_SMD:R_0201_0603Metric")
+      (reference "R5") (unit 1) (value "820") (footprint "Resistor_SMD:R_0603_1608Metric")
     )
     (path "/4f0f8793-9f3c-4eb7-ad81-220702f554ea"
-      (reference "R6") (unit 1) (value "820") (footprint "Capacitor_Tantalum_SMD:CP_EIA-7343-40_Kemet-Y")
+      (reference "R6") (unit 1) (value "820") (footprint "Resistor_SMD:R_0603_1608Metric")
     )
     (path "/00000000-0000-0000-0000-00005dfcc849"
       (reference "RLY1") (unit 1) (value "RELAY_DIL16") (footprint "custom:DIP-16_Relay")
     )
+    (path "/00000000-0000-0000-0000-00005dfd620b"
+      (reference "U1") (unit 1) (value "74HCT08") (footprint "Package_SO:SOIC-14_3.9x8.7mm_P1.27mm")
+    )
     (path "/00000000-0000-0000-0000-00005dfd0ce7"
-      (reference "U1") (unit 1) (value "74HCT08") (footprint "Package_SO:SOIC-14_3.9x8.7mm_P1.27mm")
-    )
-    (path "/00000000-0000-0000-0000-00005dfd620b"
       (reference "U1") (unit 2) (value "74HCT08") (footprint "Package_SO:SOIC-14_3.9x8.7mm_P1.27mm")
     )

Commit message: Fix bug.
Connections:
- net TH: now also J4.1 (Pin_1), J6.2 (Pin_2), R4.1, U1.4, U1.5; no longer J4.2 (Pin_2), J6.3 (Pin_3)
- new net: J4.2 (Pin_2), J6.3 (Pin_3)
Other:
- note added: "+5V"
- note added: "GND"
- note added: "H"
- note added: "NC"
- note added: "WP"
Changed lines of the file:
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@@
   (junction (at 104.14 97.79) (diameter 0) (color 0 0 0 0)
   )
-  (junction (at 48.26 76.2) (diameter 0) (color 0 0 0 0)
-  )
   (junction (at 52.07 52.07) (diameter 0) (color 0 0 0 0)
   )
@@
     (stroke (width 0) (type default) (color 0 0 0 0))
   )
-  (wire (pts (xy 48.26 69.85) (xy 48.26 76.2))
-    (stroke (width 0) (type default) (color 0 0 0 0))
-  )
   (wire (pts (xy 142.24 97.79) (xy 139.7 97.79))
     (stroke (width 0) (type default) (color 0 0 0 0))
@@
     (stroke (width 0) (type default) (color 0 0 0 0))
   )
-  (wire (pts (xy 48.26 76.2) (xy 71.12 76.2))
+  (wire (pts (xy 41.91 76.2) (xy 71.12 76.2))
     (stroke (width 0) (type default) (color 0 0 0 0))
   )
@@
     (stroke (width 0) (type default) (color 0 0 0 0))
   )
+  (wire (pts (xy 57.15 69.85) (xy 57.15 73.66))
+    (stroke (width 0) (type default) (color 0 0 0 0))
+  )
   (wire (pts (xy 160.02 107.95) (xy 177.165 107.95))
     (stroke (width 0) (type default) (color 0 0 0 0))
@@
     (stroke (width 0) (type default) (color 0 0 0 0))
   )
-  (wire (pts (xy 53.34 69.85) (xy 48.26 69.85))
-    (stroke (width 0) (type default) (color 0 0 0 0))
-  )
   (wire (pts (xy 121.92 67.31) (xy 121.92 95.25))
     (stroke (width 0) (type default) (color 0 0 0 0))
@@
     (stroke (width 0) (type default) (color 0 0 0 0))
   )
-  (wire (pts (xy 41.91 76.2) (xy 48.26 76.2))
-    (stroke (width 0) (type default) (color 0 0 0 0))
-  )
   (wire (pts (xy 153.67 64.77) (xy 153.67 67.31))
     (stroke (width 0) (type default) (color 0 0 0 0))
@@
     (stroke (width 0) (type default) (color 0 0 0 0))
   )
+  (wire (pts (xy 53.34 69.85) (xy 57.15 69.85))
+    (stroke (width 0) (type default) (color 0 0 0 0))
+  )
   (text "230 V out" (at 24.13 41.91 0)
     (effects (font (size 1.27 1.27)) (justify left bottom))
   )
+  (text "GND" (at 80.01 82.042 0)
+    (effects (font (size 1.27 1.27)) (justify left bottom))
+  )
   (text "Laser enable" (at 64.135 160.02 0)
     (effects (font (size 1.27 1.27)) (justify left bottom))
@@
     (effects (font (size 1.27 1.27)) (justify left bottom))
   )
+  (text "WP" (at 80.01 79.756 0)
+    (effects (font (size 1.27 1.27)) (justify left bottom))
+  )
   (text "230 V in" (at 24.13 62.865 0)
     (effects (font (size 1.27 1.27)) (justify left bottom))
@@
     (effects (font (size 1.27 1.27)) (justify left bottom))
   )
-  (global_label "TH" (shape input) (at 53.34 69.85 0) (fields_autoplaced)
-    (effects (font (size 1.27 1.27)) (justify left))
-    (property "Intersheet References" "${INTERSHEET_REFS}" (id 0) (at 57.9623 69.7706 0)
-      (effects (font (size 1.27 1.27)) (justify left) hide)
+  (text "+5V" (at 79.502 71.628 0)
+    (effects (font (size 1.27 1.27)) (justify left bottom))
+  )
+  (text "NC" (at 79.756 76.962 0)
+    (effects (font (size 1.27 1.27)) (justify left bottom))
+  )
+  (text "H" (at 79.756 74.422 0)
+    (effects (font (size 1.27 1.27)) (justify left bottom))
+  )
+  (global_label "TH" (shape input) (at 53.34 69.85 180) (fields_autoplaced)
+    (effects (font (size 1.27 1.27)) (justify right))
+    (property "Intersheet References" "${INTERSHEET_REFS}" (id 0) (at 48.7177 69.7706 0)
+      (effects (font (size 1.27 1.27)) (justify right) hide)
     )
   )
@@
   (symbol (lib_id "Connector_Generic:Conn_01x05") (at 76.2 76.2 0) (unit 1)
     (in_bom yes) (on_board yes)
-    (property "Reference" "J6" (id 0) (at 78.232 75.1332 0)
+    (property "Reference" "J6" (id 0) (at 74.93 84.074 0)
       (effects (font (size 1.27 1.27)) (justify left))
     )
-    (property "Value" "JST XH" (id 1) (at 78.232 77.4446 0)
+    (property "Value" "JST XH" (id 1) (at 72.39 86.36 0)
       (effects (font (size 1.27 1.27)) (justify left))
     )
