File: pcb/chillercontrol/chillercontrol.kicad_sch (KiCad schematic)
At the start: 12 parts, among them J1 PWR IN, J2 PWR OUT, J3 Switch, J4 SSR, Q1 BC547, U1 4011

Commit message: Fix bug.
Connections:
- net +24V: now also J4.1 (Pin_1)
- net at J4.2 (Pin_2): now also Q1.1 (C)
Other:
- moved on the sheet: J4
